Commit message: Ngoc commit

File: src/robot/urdf/gazebo.xacro (robot description, xacro)
@@ -8,3 +8,34 @@
         </gazebo>
     </xacro:if>
+    <link name="camera_link">
+        <visual>
+            <geometry>
+                <box size="0.05 0.05 0.05"/>
+            </geometry>
+            <material name="black"/>
+        </visual>
+    </link>
+    <joint name="camera_joint" type="fixed">
+        <parent link="world"/>
+        <child link="camera_link"/>
+        <origin xyz="0.5 0.0 1.5" rpy="0 1.57 0"/>
+    </joint>
+    <gazebo reference="camera_link">
+        <sensor name="camera" type="camera">
+            <camera>
+                <horizontal_fov>1.047</horizontal_fov>
+                <image>
+                    <width>640</width>
+                    <height>480</height>
+                </image>
+                <clip>
+                    <near>0.1</near>
+                    <far>100</far>
+                </clip>
+            </camera>
+            <always_on>1</always_on>
+            <update_rate>30</update_rate>
+            <visualize>true</visualize>
+            <topic>camera/image_raw</topic> </sensor>
+    </gazebo>
 </robot>

File: src/robot/urdf/robot.ros2_control.xacro (robot description, xacro)
@@ -7,4 +7,5 @@
                 <xacro:if value="${use_sim}">
                     <plugin>gz_ros2_control/GazeboSimSystem</plugin>
+                    <parameters>$(find robot_moveit)/config/ros2_controllers.yaml</parameters>
                 </xacro:if>
                 <xacro:unless value="${use_sim}">

File: src/robot/urdf/robot.xacro (robot description, xacro)
@@ -289,6 +289,6 @@
     <axis xyz="1 0 0" />
     <limit
-      lower="0" upper="0.02"
-      effort="1000" velocity="5.0" />
+      lower="0" upper="0.1"
+      effort="50" velocity="0.05" />
   </joint>
     <!-- gripper_r -->
@@ -325,6 +325,25 @@
     <axis xyz="1 0 0" />
     <limit
-      lower="0" upper="0.02"
-      effort="1000" velocity="5.0" />
+      lower="0" upper="0.1"
+      effort="50" velocity="0.05" />
+  </joint>
+  <gazebo reference="gripper_l">
+    <mu1>1000.0</mu1> <mu2>1000.0</mu2> <kp>1000000.0</kp> <kd>1.0</kd>       <minDepth>0.001</minDepth> <maxVel>0.1</maxVel>       <selfCollide>false</selfCollide>
+    <material>Gazebo/Grey</material>
+  </gazebo>
+  <gazebo reference="gripper_r">
+    <mu1>1000.0</mu1>
+    <mu2>1000.0</mu2>
+    <kp>1000000.0</kp>
+    <kd>1.0</kd>
+    <minDepth>0.001</minDepth>
+    <maxVel>0.1</maxVel>
+    <selfCollide>false</selfCollide>
+    <material>Gazebo/Grey</material>
+  </gazebo>
+  <link name="tcp_link"/> <joint name="tcp_joint" type="fixed">
+    <parent link="link_6"/>
+    <child link="tcp_link"/>
+    <origin xyz="0 0 0.08" rpy="0 0 0"/>
   </joint>
 </robot>
