Commit message: Astra cam xacro

File: src/robot_description/urdf/gazebo.xacro (robot description, xacro)
@@ -4,27 +4,7 @@
         <gazebo>
             <plugin filename="libgz_ros2_control-system.so" name="gz_ros2_control::GazeboSimROS2ControlPlugin">
-            <parameters>$(find robot_moveit)/config/ros2_controllers.yaml</parameters>
+                <parameters>$(find robot_moveit)/config/ros2_controllers.yaml</parameters>
             </plugin>
         </gazebo>
     </xacro:if>
-    <link name="camera_link">
-        <visual>
-            <geometry>
-                <mesh filename="package://robot_description/meshes/astra_cam.stl" />
-            </geometry>
-            <material name="black">
-                <color rgba="0 0 0 1"/>
-            </material>
-        </visual>
-        <collision>
-            <geometry>
-                <mesh filename="package://robot_description/meshes/astra_cam.stl" />
-            </geometry>
-        </collision>
-    </link>
-    <joint name="camera_joint" type="fixed">
-        <parent link="world"/>
-        <child link="camera_link"/>
-        <origin xyz="0.8 0 2" rpy="3.1416 0 1.5707"/>
-    </joint>
 </robot>

File: src/robot_description/urdf/robot.urdf.xacro (robot description, xacro)
@@ -3,7 +3,12 @@
     <xacro:arg name="use_sim" default="true" />
     <xacro:arg name="initial_positions_file" default="$(find robot_moveit)/config/initial_positions.yaml" />
-    <xacro:include filename="$(find robot_description)/urdf/robot.xacro" />
-    <xacro:include filename="$(find robot_description)/urdf/robot.ros2_control.xacro" />
-    <xacro:include filename="$(find robot_description)/urdf/gazebo.xacro" />
-    <xacro:robot_ros2_control name="robot" initial_positions_file="$(arg initial_positions_file)" use_sim="$(arg use_sim)" />
+    <xacro:include filename =   "$(find robot_description)/urdf/materials.xacro" />
+    <xacro:include filename =   "$(find robot_description)/urdf/robot.xacro" />
+    <xacro:include filename =   "$(find robot_description)/urdf/sensors.xacro"/>
+    <xacro:include filename =   "$(find robot_description)/urdf/robot.ros2_control.xacro" />
+    <xacro:include filename =   "$(find robot_description)/urdf/gazebo.xacro" />
+    <xacro:base_camera parent_link  = "base_link"/>
+    <xacro:robot_ros2_control name  ="robot"
+            initial_positions_file  ="$(arg initial_positions_file)"
+            use_sim                 ="$(arg use_sim)" />
 </robot>
